Commit message: Planning with obstacle dodge added - 18/01/17

File: golem_description/urdf/golem.xacro (robot description, xacro)
@@ -58,5 +58,5 @@
     </collision>
   </link>
-  <joint name="fixed" type="fixed">
+  <joint name="fixed_joint" type="fixed">
       <parent link="world"/>
       <child link="base_link"/>

Commit message: Motion planning test working properly

File: golem_description/urdf/golem.xacro (robot description, xacro)
@@ -14,5 +14,5 @@
     <xacro:property name="PI" value="3.1415926535897931"/>
     <xacro:property name="FRICTION" value="0.4"/>
-    <xacro:property name="JOINT_VEL" value="0.5"/>
+    <xacro:property name="JOINT_VEL" value="1.0"/>
     <xacro:property name="CONTROLLER" value="EffortJointInterface"/>
     <!-- Import all Gazebo-customization elements, including Gazebo colors -->
